File: Clicker PCB/Clicker_PCB.kicad_sch (KiCad schematic)
At the start: 47 parts, among them J1 Pogo, J2 IPX, SW1 CLICKER, SW3 BTN, SW4 BTN, U1 STM32WB07CCV6, U2 MLPF-NRG-01D3, Y1 32.768 KHz, Y2 32MHz

Commit message: Updated PCB, Beacon-Visualizer, Code Explaination, User Manual, and added back- & frontend.
Parts:
- Y1: mouser 198-XTL2024 -> 815-ABS07L-32.7-T
Connections:
- net +3V3: now also U1.32 (VFBSD), U1.36 (VDDSD)
- no-connect marks 11 -> 9
Other:
- note added: "These are left floating in the V1 PCB!"
Changed lines of the file:
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@@
 	)
 	(junction
+		(at 85.09 57.15)
+		(diameter 0)
+		(color 0 0 0 0)
+	)
+	(junction
 		(at 67.31 45.72)
 		(diameter 0)
@@
 	)
 	(no_connect
-		(at 82.55 57.15)
-	)
-	(no_connect
 		(at 44.45 88.9)
 	)
@@
 	)
 	(no_connect
-		(at 82.55 59.69)
-	)
-	(no_connect
 		(at 82.55 93.98)
 	)
@@
 	(wire
 		(pts
+			(xy 85.09 59.69) (xy 85.09 57.15)
+		)
+		(stroke
+			(width 0)
+			(type default)
+		)
+	)
+	(wire
+		(pts
+			(xy 82.55 59.69) (xy 85.09 59.69)
+		)
+		(stroke
+			(width 0)
+			(type default)
+		)
+	)
+	(wire
+		(pts
 			(xy 132.08 100.33) (xy 133.35 100.33)
 		)
@@
 	(wire
 		(pts
+			(xy 82.55 57.15) (xy 85.09 57.15)
+		)
+		(stroke
+			(width 0)
+			(type default)
+		)
+	)
+	(wire
+		(pts
 			(xy 127 182.88) (xy 127 181.61)
 		)
@@
 	(wire
 		(pts
+			(xy 85.09 57.15) (xy 85.09 54.61)
+		)
+		(stroke
+			(width 0)
+			(type default)
+		)
+	)
+	(wire
+		(pts
 			(xy 64.77 119.38) (xy 64.77 118.11)
 		)
@@
 		)
 	)
+	(text "These are left floating\nin the V1 PCB!"
+		(exclude_from_sim no)
+		(at 96.52 49.53 0)
+		(effects
+			(font
+				(size 1.27 1.27)
+			)
+		)
+	)
 	(text "LED"
 		(exclude_from_sim no)
@@
 	)
 	(symbol
+		(lib_id "power:+3V3")
+		(at 85.09 54.61 0)
+		(unit 1)
+		(exclude_from_sim no)
+		(in_bom yes)
+		(on_board yes)
+		(dnp no)
+		(property "Reference" "#PWR09"
+			(at 85.09 58.42 0)
+			(effects
+				(font
+					(size 1.27 1.27)
+				)
+				(hide yes)
+			)
+		)
+		(property "Value" "+3V3"
+			(at 85.09 50.8 0)
+			(effects
+				(font
+					(size 1.27 1.27)
+				)
+			)
+		)
+		(property "Footprint" ""
+			(at 85.09 54.61 0)
+			(effects
+				(font
+					(size 1.27 1.27)
+				)
+				(hide yes)
+			)
+		)
+		(property "Datasheet" ""
+			(at 85.09 54.61 0)
+			(effects
+				(font
+					(size 1.27 1.27)
+				)
+				(hide yes)
+			)
+		)
+		(property "Description" "Power symbol creates a global label with name \"+3V3\""
+			(at 85.09 54.61 0)
+			(effects
+				(font
+					(size 1.27 1.27)
+				)
+				(hide yes)
+			)
+		)
+		(pin "1"
+		)
+		(instances
+			(project "Clicker_PCB"
+				(path "/74379efc-e377-48e5-ad16-86adc14a8363"
+					(reference "#PWR09")
+					(unit 1)
+				)
+			)
+		)
+	)
+	(symbol
 		(lib_id "power:GND")
 		(at 120.65 109.22 0)
@@
 			)
 		)
-		(property "mouser" " 198-XTL2024"
+		(property "mouser" "815-ABS07L-32.7-T"
 			(at 160.02 180.34 0)
 			(effects
