File: Clicker PCB/PWR.kicad_sch (KiCad schematic)
At the start: 22 parts, among them U3 MCP73833, U4 ISL91127IR

Commit message: Updated PCB, Beacon-Visualizer, Code Explaination, User Manual, and added back- & frontend.
Parts:
- F1: mouser 504-PTS18126V125 -> 504-PTS18126V260
Changed lines of the file:
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@@
 			)
 		)
-		(property "mouser" " 504-PTS18126V125"
+		(property "mouser" "504-PTS18126V260"
 			(at 33.02 35.56 0)
 			(effects
