File: Clicker PCB/UWB.kicad_sch (KiCad schematic)
At the start: 53 parts, among them U5 DW1000, U6 LXDC2HL18A-052, U7 HHM1595A1, Y3 38.4MHz

Commit message: Updated PCB, Beacon-Visualizer, Code Explaination, User Manual, and added back- & frontend.
Parts:
- C35, U6: now not fitted
- R20: now fitted
Changed lines of the file:
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@@
 		(in_bom yes)
 		(on_board yes)
-		(dnp yes)
+		(dnp no)
 		(property "Reference" "R20"
 			(at 49.022 139.7 90)
@@
 		(in_bom yes)
 		(on_board yes)
-		(dnp no)
+		(dnp yes)
 		(property "Reference" "C35"
 			(at 26.416 146.812 0)
@@
 		(in_bom yes)
 		(on_board yes)
-		(dnp no)
+		(dnp yes)
 		(property "Reference" "U6"
 			(at 40.64 147.32 0)
